File: electronics/nff_pcb/a33_power.kicad_sch (KiCad schematic)
At the start: 25 parts, among them U2 A33

Commit message: R0.1 released.
Parts:
- C53, C54, C55, C56, C69, C70: MPN GRM155R60J226ME11D -> GRM158R60J226ME01D
- U2: MPN A33 -> "Allwinner A33" or "Allwinner R16"
Changed lines of the file:
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@@
 			)
 		)
-		(property "MPN" "GRM155R60J226ME11D"
+		(property "MPN" "GRM158R60J226ME01D"
 			(at 95.25 100.33 0)
 			(effects
@@
 			)
 		)
-		(property "MPN" "GRM155R60J226ME11D"
+		(property "MPN" "GRM158R60J226ME01D"
 			(at 95.25 43.18 0)
 			(effects
@@
 			)
 		)
-		(property "MPN" "GRM155R60J226ME11D"
+		(property "MPN" "GRM158R60J226ME01D"
 			(at 142.24 127 0)
 			(effects
@@
 			)
 		)
-		(property "MPN" "GRM155R60J226ME11D"
+		(property "MPN" "GRM158R60J226ME01D"
 			(at 92.71 73.66 0)
 			(effects
@@
 			)
 		)
-		(property "MPN" "GRM155R60J226ME11D"
+		(property "MPN" "GRM158R60J226ME01D"
 			(at 140.97 100.33 0)
 			(effects
@@
 			)
 		)
-		(property "MPN" "GRM155R60J226ME11D"
+		(property "MPN" "GRM158R60J226ME01D"
 			(at 100.33 127 0)
 			(effects
@@
 			)
 		)
-		(property "MPN" "A33"
+		(property "MPN" "\"Allwinner A33\" or \"Allwinner R16\""
 			(at 191.77 32.639 0)
 			(effects
