File: electronics/nff_pcb/a33_ram.kicad_sch (KiCad schematic)
At the start: 8 parts, among them U2 A33

Commit message: R0.1 released.
Parts:
- U2: MPN A33 -> "Allwinner A33" or "Allwinner R16"
Changed lines of the file:
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@@
 			)
 		)
-		(property "MPN" "A33"
+		(property "MPN" "\"Allwinner A33\" or \"Allwinner R16\""
 			(at 151.13 46.609 0)
 			(effects
