File: electronics/nff_pcb/dsi.kicad_sch (KiCad schematic)
At the start: 8 parts, among them J8 Conn_01x20_MountingPin, U9 AP3036B

Commit message: R0.1 released.
Parts:
- C34: footprint Capacitor_SMD:C_0603_1608Metric -> Capacitor_SMD:C_0402_1005Metric; MPN (none) -> CL05A105KO5NNNC
- C35: MPN (none) -> CC0603KRX7R7BB224
- U9: MPN (none) -> AP3036BKTR-G1
Changed lines of the file:
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@@
+			)
+		)
+		(property "MPN" "CC0603KRX7R7BB224"
+			(at 163.83 53.34 0)
+			(effects
+				(font
+					(size 1.27 1.27)
+				)
+				(hide yes)
 			)
 		)
@@
 			)
 		)
+		(property "MPN" "AP3036BKTR-G1"
+			(at 134.62 60.96 0)
+			(effects
+				(font
+					(size 1.27 1.27)
+				)
+				(hide yes)
+			)
+		)
 		(pin "1"
 		)
@@
 			)
 		)
-		(property "Footprint" "Capacitor_SMD:C_0603_1608Metric"
+		(property "Footprint" "Capacitor_SMD:C_0402_1005Metric"
 			(at 120.65 48.26 0)
 			(effects
@@
 			(at 120.65 48.26 0)
 			(effects
+				(font
+					(size 1.27 1.27)
+				)
+				(hide yes)
+			)
+		)
+		(property "MPN" "CL05A105KO5NNNC"
+			(at 120.65 48.26 0)
+			(effects
