File: electronics/nff_pcb/ram.kicad_sch (KiCad schematic)
At the start: 23 parts, among them U1 AS4C512M16D3L-12BIN

Commit message: R2 Released
Parts:
- U1: MPN AS4C512M16D3L-12BIN -> ZDV4256M16A-13DPH
Other:
- note added: "DDR3L 96Pin BGA"
- note added: "OG Part AS4C512M16D3L-12BIN"
Changed lines of the file:
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@@
+		)
+	)
+	(text "OG Part\nAS4C512M16D3L-12BIN"
+		(exclude_from_sim no)
+		(at 103.378 35.052 0)
+		(effects
+			(font
+				(size 1.27 1.27)
+			)
+		)
+	)
+	(text "DDR3L\n96Pin BGA"
+		(exclude_from_sim no)
+		(at 107.95 24.384 0)
+		(effects
+			(font
+				(size 4 4)
+			)
 		)
 	)
@@
 			)
 		)
-		(property "MPN" "AS4C512M16D3L-12BIN"
+		(property "MPN" "ZDV4256M16A-13DPH"
 			(at 226.06 45.339 0)
 			(effects
@@
 			)
 		)
-		(property "MPN" "AS4C512M16D3L-12BIN"
+		(property "MPN" "ZDV4256M16A-13DPH"
 			(at 44.45 31.75 0)
 			(effects
