File: electronics/nff_pcb/wifi.kicad_sch (KiCad schematic)
At the start: 20 parts, among them J7 Conn_Coaxial, U8 RTL8723DS

Commit message: R0.1 released.
Parts:
- L5: MPN (none) -> BLM18KG121TN1D
- R35: MPN RC0402FR-130RL -> RC0402FR-070RL
Connections:
- net CLK renamed SDC1.CLK
- net CMD renamed SDC1.CMD
- net D0 renamed SDC1.D0
- net D1 renamed SDC1.D1
- net D2 renamed SDC1.D2
- net D3 renamed SDC1.D3
Changed lines of the file:
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@@
 		(members "WAKE" "HOST_WAKE" "RST_N")
 	)
-	(bus_alias "SDC"
-		(members "D[3..0]" "CLK" "CMD")
+	(bus_alias "SDC1"
+		(members "SDC1.D[3..0]" "SDC1.CLK" "SDC1.CMD")
 	)
 	(bus_alias "UART"
@@
 	)
 	(junction
-		(at 162.56 68.58)
-		(diameter 0)
-		(color 0 0 0 0)
-	)
-	(junction
 		(at 162.56 132.08)
 		(diameter 0)
@@
 	(wire
 		(pts
-			(xy 160.02 66.04) (xy 162.56 66.04)
+			(xy 160.02 66.04) (xy 163.83 66.04)
 		)
 		(stroke
@@
 	(wire
 		(pts
-			(xy 162.56 68.58) (xy 162.56 66.04)
+			(xy 163.83 68.58) (xy 163.83 66.04)
 		)
 		(stroke
@@
 		)
 	)
-	(wire
-		(pts
-			(xy 162.56 68.58) (xy 163.83 68.58)
-		)
-		(stroke
-			(width 0)
-			(type default)
-		)
-	)
 	(bus
 		(pts
@@
 	(wire
 		(pts
-			(xy 157.48 68.58) (xy 162.56 68.58)
+			(xy 157.48 68.58) (xy 163.83 68.58)
 		)
 		(stroke
@@
 		)
 	)
-	(label "D0"
+	(label "SDC1.D0"
 		(at 72.39 81.28 0)
 		(fields_autoplaced yes)
@@
 		)
 	)
-	(label "CLK"
+	(label "SDC1.CLK"
 		(at 72.39 78.74 0)
 		(fields_autoplaced yes)
@@
 		)
 	)
-	(label "CMD"
+	(label "SDC1.CMD"
 		(at 72.39 76.2 0)
 		(fields_autoplaced yes)
@@
 		)
 	)
-	(label "D3"
+	(label "SDC1.D3"
 		(at 72.39 73.66 0)
 		(fields_autoplaced yes)
@@
 		)
 	)
-	(label "D1"
+	(label "SDC1.D1"
 		(at 72.39 83.82 0)
 		(fields_autoplaced yes)
@@
 		)
 	)
-	(label "D2"
+	(label "SDC1.D2"
 		(at 72.39 71.12 0)
 		(fields_autoplaced yes)
@@
 		)
 	)
-	(hierarchical_label "{SDC}"
+	(hierarchical_label "{SDC1}"
 		(shape input)
 		(at 64.77 59.69 180)
@@
 			)
 		)
-		(property "MPN" "RC0402FR-130RL"
+		(property "MPN" "RC0402FR-070RL"
 			(at 104.14 127 90)
 			(effects
@@
 			)
 		)
-		(property "MPN" ""
+		(property "MPN" "BLM18KG121TN1D"
 			(at 205.74 71.12 90)
 			(effects

Commit message: Added the proper SMA conntector
Parts:
- J7: MPN 901-143-6RFX -> CONREVSMA002-G
Changed lines of the file:
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@@
 			)
 		)
-		(property "MPN" "901-143-6RFX"
+		(property "MPN" "CONREVSMA002-G"
 			(at 85.09 127 0)
 			(effects

Commit message: R2 Released
Parts:
- J7: MPN CONREVSMA002-G -> SMA-KWE901
- R33, R36: MPN RC0402FR-131KL -> RC0402JR-071KL
- R37: value 100K -> 100k
- R39: MPN RC0402FR-1310KL -> RC0402JR-0710KL
Changed lines of the file:
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@@
 			)
 		)
-		(property "MPN" "RC0402FR-131KL"
+		(property "MPN" "RC0402JR-071KL"
 			(at 110.49 106.68 90)
 			(effects
@@
 			)
 		)
-		(property "Datasheet" " ~"
+		(property "Datasheet" "~"
 			(at 85.09 127 0)
 			(effects
@@
 			)
 		)
-		(property "MPN" "CONREVSMA002-G"
+		(property "MPN" "SMA-KWE901"
 			(at 85.09 127 0)
 			(effects
@@
 			)
 		)
-		(property "MPN" "RC0402FR-131KL"
+		(property "MPN" "RC0402JR-071KL"
 			(at 101.6 104.14 90)
 			(effects
@@
 			)
 		)
-		(property "MPN" "RC0402FR-1310KL"
+		(property "MPN" "RC0402JR-0710KL"
 			(at 184.15 95.25 0)
 			(effects
@@
 			)
 		)
-		(property "Value" "100K"
+		(property "Value" "100k"
 			(at 171.45 111.125 0)
 			(effects
